Commit message: renaming instances of drc robot to atlas

File: models/drc_robot/model.urdf (robot description, URDF)
Before this commit: robot drc_robot, 40 links, 39 joints
Links:
- link l_clav: geometry collision mesh filename=package://atlas/meshes/l_clav.stl scale=1 1 1; visual mesh filename=package://atlas/meshes/l_clav.dae scale=1 1 1
- link l_farm: geometry collision mesh filename=package://atlas/meshes/l_farm.stl scale=1 1 1; visual mesh filename=package://atlas/meshes/l_farm.dae scale=1 1 1
- link l_foot: geometry collision mesh filename=package://atlas/meshes/l_foot.stl scale=1 1 1; visual mesh filename=package://atlas/meshes/l_foot.dae scale=1 1 1
- link l_hand: geometry collision mesh filename=package://atlas/meshes/l_hand.stl scale=1 1 1; visual mesh filename=package://atlas/meshes/l_hand.dae scale=1 1 1
- link l_larm: geometry collision mesh filename=package://atlas/meshes/l_larm.stl scale=1 1 1; visual mesh filename=package://atlas/meshes/l_larm.dae scale=1 1 1
- link l_lglut: geometry collision mesh filename=package://atlas/meshes/l_lglut.stl scale=1 1 1; visual mesh filename=package://atlas/meshes/l_lglut.dae scale=1 1 1
- link l_lleg: geometry collision mesh filename=package://atlas/meshes/l_lleg.stl scale=1 1 1; visual mesh filename=package://atlas/meshes/l_lleg.dae scale=1 1 1
- link l_scap: geometry collision mesh filename=package://atlas/meshes/l_scap.stl scale=1 1 1; visual mesh filename=package://atlas/meshes/l_scap.dae scale=1 1 1
- link l_talus: geometry collision mesh filename=package://atlas/meshes/l_talus.stl scale=1 1 1; visual mesh filename=package://atlas/meshes/l_talus.dae scale=1 1 1
- link l_uarm: geometry collision mesh filename=package://atlas/meshes/l_uarm.stl scale=1 1 1; visual mesh filename=package://atlas/meshes/l_uarm.dae scale=1 1 1
- link l_uglut: geometry collision mesh filename=package://atlas/meshes/l_uglut.stl scale=1 1 1; visual mesh filename=package://atlas/meshes/l_uglut.dae scale=1 1 1
- link l_uleg: geometry collision mesh filename=package://atlas/meshes/l_uleg.stl scale=1 1 1; visual mesh filename=package://atlas/meshes/l_uleg.dae scale=1 1 1
- link ltorso: geometry collision mesh filename=package://atlas/meshes/ltorso.stl scale=1 1 1; visual mesh filename=package://atlas/meshes/ltorso.dae scale=1 1 1
- link mtorso: geometry collision mesh filename=package://atlas/meshes/mtorso.stl scale=1 1 1; visual mesh filename=package://atlas/meshes/mtorso.dae scale=1 1 1
- link pelvis: geometry collision mesh filename=package://atlas/meshes/pelvis.stl scale=1 1 1; visual mesh filename=package://atlas/meshes/pelvis.dae scale=1 1 1
- link r_clav: geometry collision mesh filename=package://atlas/meshes/r_clav.stl scale=1 1 1; visual mesh filename=package://atlas/meshes/r_clav.dae scale=1 1 1
- link r_farm: geometry collision mesh filename=package://atlas/meshes/r_farm.stl scale=1 1 1; visual mesh filename=package://atlas/meshes/r_farm.dae scale=1 1 1
- link r_foot: geometry collision mesh filename=package://atlas/meshes/r_foot.stl scale=1 1 1; visual mesh filename=package://atlas/meshes/r_foot.dae scale=1 1 1
- link r_hand: geometry collision mesh filename=package://atlas/meshes/r_hand.stl scale=1 1 1; visual mesh filename=package://atlas/meshes/r_hand.dae scale=1 1 1
- link r_larm: geometry collision mesh filename=package://atlas/meshes/r_larm.stl scale=1 1 1; visual mesh filename=package://atlas/meshes/r_larm.dae scale=1 1 1
- link r_lglut: geometry collision mesh filename=package://atlas/meshes/r_lglut.stl scale=1 1 1; visual mesh filename=package://atlas/meshes/r_lglut.dae scale=1 1 1
- link r_lleg: geometry collision mesh filename=package://atlas/meshes/r_lleg.stl scale=1 1 1; visual mesh filename=package://atlas/meshes/r_lleg.dae scale=1 1 1
- link r_scap: geometry collision mesh filename=package://atlas/meshes/r_scap.stl scale=1 1 1; visual mesh filename=package://atlas/meshes/r_scap.dae scale=1 1 1
- link r_talus: geometry collision mesh filename=package://atlas/meshes/r_talus.stl scale=1 1 1; visual mesh filename=package://atlas/meshes/r_talus.dae scale=1 1 1
- link r_uarm: geometry collision mesh filename=package://atlas/meshes/r_uarm.stl scale=1 1 1; visual mesh filename=package://atlas/meshes/r_uarm.dae scale=1 1 1
- link r_uglut: geometry collision mesh filename=package://atlas/meshes/r_uglut.stl scale=1 1 1; visual mesh filename=package://atlas/meshes/r_uglut.dae scale=1 1 1
- link r_uleg: geometry collision mesh filename=package://atlas/meshes/r_uleg.stl scale=1 1 1; visual mesh filename=package://atlas/meshes/r_uleg.dae scale=1 1 1
- link utorso: geometry collision mesh filename=package://atlas/meshes/utorso.stl scale=1 1 1; visual mesh filename=package://atlas/meshes/utorso.dae scale=1 1 1

File: models/drc_robot_irobot_hand/model.urdf (robot description, URDF)
Before this commit: robot drc_robot, 101 links, 100 joints
Links:
- link head: geometry collision mesh filename=package://atlas/meshes/head.stl scale=1 1 1; visual mesh filename=package://atlas/meshes/head.dae scale=1 1 1
- link l_clav: geometry collision mesh filename=package://atlas/meshes/l_clav.stl scale=1 1 1; visual mesh filename=package://atlas/meshes/l_clav.dae scale=1 1 1
- link l_farm: geometry collision mesh filename=package://atlas/meshes/l_farm.stl scale=1 1 1; visual mesh filename=package://atlas/meshes/l_farm.dae scale=1 1 1
- link l_foot: geometry collision mesh filename=package://atlas/meshes/l_foot.stl scale=1 1 1; visual mesh filename=package://atlas/meshes/l_foot.dae scale=1 1 1
- link l_hand: geometry collision mesh filename=package://atlas/meshes/l_hand.stl scale=1 1 1; visual mesh filename=package://atlas/meshes/l_hand.dae scale=1 1 1
- link l_larm: geometry collision mesh filename=package://atlas/meshes/l_larm.stl scale=1 1 1; visual mesh filename=package://atlas/meshes/l_larm.dae scale=1 1 1
- link l_lglut: geometry collision mesh filename=package://atlas/meshes/l_lglut.stl scale=1 1 1; visual mesh filename=package://atlas/meshes/l_lglut.dae scale=1 1 1
- link l_lleg: geometry collision mesh filename=package://atlas/meshes/l_lleg.stl scale=1 1 1; visual mesh filename=package://atlas/meshes/l_lleg.dae scale=1 1 1
- link l_scap: geometry collision mesh filename=package://atlas/meshes/l_scap.stl scale=1 1 1; visual mesh filename=package://atlas/meshes/l_scap.dae scale=1 1 1
- link l_talus: geometry collision mesh filename=package://atlas/meshes/l_talus.stl scale=1 1 1; visual mesh filename=package://atlas/meshes/l_talus.dae scale=1 1 1
- link l_uarm: geometry collision mesh filename=package://atlas/meshes/l_uarm.stl scale=1 1 1; visual mesh filename=package://atlas/meshes/l_uarm.dae scale=1 1 1
- link l_uglut: geometry collision mesh filename=package://atlas/meshes/l_uglut.stl scale=1 1 1; visual mesh filename=package://atlas/meshes/l_uglut.dae scale=1 1 1
- link l_uleg: geometry collision mesh filename=package://atlas/meshes/l_uleg.stl scale=1 1 1; visual mesh filename=package://atlas/meshes/l_uleg.dae scale=1 1 1
- link ltorso: geometry collision mesh filename=package://atlas/meshes/ltorso.stl scale=1 1 1; visual mesh filename=package://atlas/meshes/ltorso.dae scale=1 1 1
- link mtorso: geometry collision mesh filename=package://atlas/meshes/mtorso.stl scale=1 1 1; visual mesh filename=package://atlas/meshes/mtorso.dae scale=1 1 1
- link pelvis: geometry collision mesh filename=package://atlas/meshes/pelvis.stl scale=1 1 1; visual mesh filename=package://atlas/meshes/pelvis.dae scale=1 1 1
- link r_clav: geometry collision mesh filename=package://atlas/meshes/r_clav.stl scale=1 1 1; visual mesh filename=package://atlas/meshes/r_clav.dae scale=1 1 1
- link r_farm: geometry collision mesh filename=package://atlas/meshes/r_farm.stl scale=1 1 1; visual mesh filename=package://atlas/meshes/r_farm.dae scale=1 1 1
- link r_foot: geometry collision mesh filename=package://atlas/meshes/r_foot.stl scale=1 1 1; visual mesh filename=package://atlas/meshes/r_foot.dae scale=1 1 1
- link r_hand: geometry collision mesh filename=package://atlas/meshes/r_hand.stl scale=1 1 1; visual mesh filename=package://atlas/meshes/r_hand.dae scale=1 1 1
- link r_larm: geometry collision mesh filename=package://atlas/meshes/r_larm.stl scale=1 1 1; visual mesh filename=package://atlas/meshes/r_larm.dae scale=1 1 1
- link r_lglut: geometry collision mesh filename=package://atlas/meshes/r_lglut.stl scale=1 1 1; visual mesh filename=package://atlas/meshes/r_lglut.dae scale=1 1 1
- link r_lleg: geometry collision mesh filename=package://atlas/meshes/r_lleg.stl scale=1 1 1; visual mesh filename=package://atlas/meshes/r_lleg.dae scale=1 1 1
- link r_scap: geometry collision mesh filename=package://atlas/meshes/r_scap.stl scale=1 1 1; visual mesh filename=package://atlas/meshes/r_scap.dae scale=1 1 1
- link r_talus: geometry collision mesh filename=package://atlas/meshes/r_talus.stl scale=1 1 1; visual mesh filename=package://atlas/meshes/r_talus.dae scale=1 1 1
- link r_uarm: geometry collision mesh filename=package://atlas/meshes/r_uarm.stl scale=1 1 1; visual mesh filename=package://atlas/meshes/r_uarm.dae scale=1 1 1
- link r_uglut: geometry collision mesh filename=package://atlas/meshes/r_uglut.stl scale=1 1 1; visual mesh filename=package://atlas/meshes/r_uglut.dae scale=1 1 1
- link r_uleg: geometry collision mesh filename=package://atlas/meshes/r_uleg.stl scale=1 1 1; visual mesh filename=package://atlas/meshes/r_uleg.dae scale=1 1 1
- link utorso: geometry collision mesh filename=package://atlas/meshes/utorso.stl scale=1 1 1; visual mesh filename=package://atlas/meshes/utorso.dae scale=1 1 1

File: models/drc_robot_sandia_hand/model.urdf (robot description, URDF)
Before this commit: robot drc_robot, 93 links, 92 joints
Links:
- link head: geometry collision mesh filename=package://atlas/meshes/head.stl scale=1 1 1; visual mesh filename=package://atlas/meshes/head.dae scale=1 1 1
- link l_clav: geometry collision mesh filename=package://atlas/meshes/l_clav.stl scale=1 1 1; visual mesh filename=package://atlas/meshes/l_clav.dae scale=1 1 1
- link l_farm: geometry collision mesh filename=package://atlas/meshes/l_farm.stl scale=1 1 1; visual mesh filename=package://atlas/meshes/l_farm.dae scale=1 1 1
- link l_foot: geometry collision mesh filename=package://atlas/meshes/l_foot.stl scale=1 1 1; visual mesh filename=package://atlas/meshes/l_foot.dae scale=1 1 1
- link l_hand: geometry collision mesh filename=package://atlas/meshes/l_hand.stl scale=1 1 1; visual mesh filename=package://atlas/meshes/l_hand.dae scale=1 1 1
- link l_larm: geometry collision mesh filename=package://atlas/meshes/l_larm.stl scale=1 1 1; visual mesh filename=package://atlas/meshes/l_larm.dae scale=1 1 1
- link l_lglut: geometry collision mesh filename=package://atlas/meshes/l_lglut.stl scale=1 1 1; visual mesh filename=package://atlas/meshes/l_lglut.dae scale=1 1 1
- link l_lleg: geometry collision mesh filename=package://atlas/meshes/l_lleg.stl scale=1 1 1; visual mesh filename=package://atlas/meshes/l_lleg.dae scale=1 1 1
- link l_scap: geometry collision mesh filename=package://atlas/meshes/l_scap.stl scale=1 1 1; visual mesh filename=package://atlas/meshes/l_scap.dae scale=1 1 1
- link l_talus: geometry collision mesh filename=package://atlas/meshes/l_talus.stl scale=1 1 1; visual mesh filename=package://atlas/meshes/l_talus.dae scale=1 1 1
- link l_uarm: geometry collision mesh filename=package://atlas/meshes/l_uarm.stl scale=1 1 1; visual mesh filename=package://atlas/meshes/l_uarm.dae scale=1 1 1
- link l_uglut: geometry collision mesh filename=package://atlas/meshes/l_uglut.stl scale=1 1 1; visual mesh filename=package://atlas/meshes/l_uglut.dae scale=1 1 1
- link l_uleg: geometry collision mesh filename=package://atlas/meshes/l_uleg.stl scale=1 1 1; visual mesh filename=package://atlas/meshes/l_uleg.dae scale=1 1 1
- link ltorso: geometry collision mesh filename=package://atlas/meshes/ltorso.stl scale=1 1 1; visual mesh filename=package://atlas/meshes/ltorso.dae scale=1 1 1
- link mtorso: geometry collision mesh filename=package://atlas/meshes/mtorso.stl scale=1 1 1; visual mesh filename=package://atlas/meshes/mtorso.dae scale=1 1 1
- link pelvis: geometry collision mesh filename=package://atlas/meshes/pelvis.stl scale=1 1 1; visual mesh filename=package://atlas/meshes/pelvis.dae scale=1 1 1
- link r_clav: geometry collision mesh filename=package://atlas/meshes/r_clav.stl scale=1 1 1; visual mesh filename=package://atlas/meshes/r_clav.dae scale=1 1 1
- link r_farm: geometry collision mesh filename=package://atlas/meshes/r_farm.stl scale=1 1 1; visual mesh filename=package://atlas/meshes/r_farm.dae scale=1 1 1
- link r_foot: geometry collision mesh filename=package://atlas/meshes/r_foot.stl scale=1 1 1; visual mesh filename=package://atlas/meshes/r_foot.dae scale=1 1 1
- link r_hand: geometry collision mesh filename=package://atlas/meshes/r_hand.stl scale=1 1 1; visual mesh filename=package://atlas/meshes/r_hand.dae scale=1 1 1
- link r_larm: geometry collision mesh filename=package://atlas/meshes/r_larm.stl scale=1 1 1; visual mesh filename=package://atlas/meshes/r_larm.dae scale=1 1 1
- link r_lglut: geometry collision mesh filename=package://atlas/meshes/r_lglut.stl scale=1 1 1; visual mesh filename=package://atlas/meshes/r_lglut.dae scale=1 1 1
- link r_lleg: geometry collision mesh filename=package://atlas/meshes/r_lleg.stl scale=1 1 1; visual mesh filename=package://atlas/meshes/r_lleg.dae scale=1 1 1
- link r_scap: geometry collision mesh filename=package://atlas/meshes/r_scap.stl scale=1 1 1; visual mesh filename=package://atlas/meshes/r_scap.dae scale=1 1 1
- link r_talus: geometry collision mesh filename=package://atlas/meshes/r_talus.stl scale=1 1 1; visual mesh filename=package://atlas/meshes/r_talus.dae scale=1 1 1
- link r_uarm: geometry collision mesh filename=package://atlas/meshes/r_uarm.stl scale=1 1 1; visual mesh filename=package://atlas/meshes/r_uarm.dae scale=1 1 1
- link r_uglut: geometry collision mesh filename=package://atlas/meshes/r_uglut.stl scale=1 1 1; visual mesh filename=package://atlas/meshes/r_uglut.dae scale=1 1 1
- link r_uleg: geometry collision mesh filename=package://atlas/meshes/r_uleg.stl scale=1 1 1; visual mesh filename=package://atlas/meshes/r_uleg.dae scale=1 1 1
- link utorso: geometry collision mesh filename=package://atlas/meshes/utorso.stl scale=1 1 1; visual mesh filename=package://atlas/meshes/utorso.dae scale=1 1 1

File: ros/drc_robot_utils/robots/drc_robot.model.xacro (robot description, xacro)
@@ -3,8 +3,8 @@
        xmlns:interface="http://playerstage.sourceforge.net/gazebo/xmlschema/#interface"
        xmlns:xacro="http://playerstage.sourceforge.net/gazebo/xmlschema/#interface"
-       name="drc_robot" >
-  <include filename="$(find drc_robot_utils)/urdf/drc_robot.urdf" />
-  <include filename="$(find drc_robot_utils)/urdf/drc_robot.gazebo" />
-  <include filename="$(find drc_robot_utils)/urdf/drc_robot.transmission" />
-  <include filename="$(find drc_robot_utils)/urdf/drc_robot.sensors" />
+       name="atlas" >
+  <include filename="$(find atlas_utils)/urdf/atlas.urdf" />
+  <include filename="$(find atlas_utils)/urdf/atlas.gazebo" />
+  <include filename="$(find atlas_utils)/urdf/atlas.transmission" />
+  <include filename="$(find atlas_utils)/urdf/atlas.sensors" />
 </robot>

File: ros/drc_robot_utils/robots/drc_robot_sandia_hands.model.xacro (robot description, xacro)
@@ -3,6 +3,6 @@
        xmlns:interface="http://playerstage.sourceforge.net/gazebo/xmlschema/#interface"
        xmlns:xacro="http://playerstage.sourceforge.net/gazebo/xmlschema/#interface"
-       name="drc_robot" >
-  <include filename="$(find drc_robot_utils)/urdf/drc_robot.urdf" />
+       name="atlas" >
+  <include filename="$(find atlas_utils)/urdf/atlas.urdf" />
   <include filename="$(find sandia_hand_utils)/urdf/sandia_hand.urdf.xacro" />
   <xacro:sandia_hand side="r" parent="r_hand">
@@ -12,6 +12,6 @@
     <origin xyz="0  0.1 -0.03" rpy="0 3.1416 -1.57079"/>
   </xacro:sandia_hand>
-  <include filename="$(find drc_robot_utils)/urdf/drc_robot.gazebo" />
-  <include filename="$(find drc_robot_utils)/urdf/drc_robot.transmission" />
-  <include filename="$(find drc_robot_utils)/urdf/drc_robot.sensors" />
+  <include filename="$(find atlas_utils)/urdf/atlas.gazebo" />
+  <include filename="$(find atlas_utils)/urdf/atlas.transmission" />
+  <include filename="$(find atlas_utils)/urdf/atlas.sensors" />
 </robot>

File: ros/drc_robot_utils/urdf/drc_robot.urdf (robot description, URDF)
Before this commit: robot drc_skeleton, 29 links, 28 joints
Links:
- link head: geometry collision mesh filename=package://atlas/meshes/head.stl scale=1 1 1; visual mesh filename=package://atlas/meshes/head.dae scale=1 1 1
- link l_clav: geometry collision mesh filename=package://atlas/meshes/l_clav.stl scale=1 1 1; visual mesh filename=package://atlas/meshes/l_clav.dae scale=1 1 1
- link l_farm: geometry collision mesh filename=package://atlas/meshes/l_farm.stl scale=1 1 1; visual mesh filename=package://atlas/meshes/l_farm.dae scale=1 1 1
- link l_foot: geometry collision mesh filename=package://atlas/meshes/l_foot.stl scale=1 1 1; visual mesh filename=package://atlas/meshes/l_foot.dae scale=1 1 1
- link l_hand: geometry collision mesh filename=package://atlas/meshes/l_hand.stl scale=1 1 1; visual mesh filename=package://atlas/meshes/l_hand.dae scale=1 1 1
- link l_larm: geometry collision mesh filename=package://atlas/meshes/l_larm.stl scale=1 1 1; visual mesh filename=package://atlas/meshes/l_larm.dae scale=1 1 1
- link l_lglut: geometry collision mesh filename=package://atlas/meshes/l_lglut.stl scale=1 1 1; visual mesh filename=package://atlas/meshes/l_lglut.dae scale=1 1 1
- link l_lleg: geometry collision mesh filename=package://atlas/meshes/l_lleg.stl scale=1 1 1; visual mesh filename=package://atlas/meshes/l_lleg.dae scale=1 1 1
- link l_scap: geometry collision mesh filename=package://atlas/meshes/l_scap.stl scale=1 1 1; visual mesh filename=package://atlas/meshes/l_scap.dae scale=1 1 1
- link l_talus: geometry collision mesh filename=package://atlas/meshes/l_talus.stl scale=1 1 1; visual mesh filename=package://atlas/meshes/l_talus.dae scale=1 1 1
- link l_uarm: geometry collision mesh filename=package://atlas/meshes/l_uarm.stl scale=1 1 1; visual mesh filename=package://atlas/meshes/l_uarm.dae scale=1 1 1
- link l_uglut: geometry collision mesh filename=package://atlas/meshes/l_uglut.stl scale=1 1 1; visual mesh filename=package://atlas/meshes/l_uglut.dae scale=1 1 1
- link l_uleg: geometry collision mesh filename=package://atlas/meshes/l_uleg.stl scale=1 1 1; visual mesh filename=package://atlas/meshes/l_uleg.dae scale=1 1 1
- link ltorso: geometry collision mesh filename=package://atlas/meshes/ltorso.stl scale=1 1 1; visual mesh filename=package://atlas/meshes/ltorso.dae scale=1 1 1
- link mtorso: geometry collision mesh filename=package://atlas/meshes/mtorso.stl scale=1 1 1; visual mesh filename=package://atlas/meshes/mtorso.dae scale=1 1 1
- link pelvis: geometry collision mesh filename=package://atlas/meshes/pelvis.stl scale=1 1 1; visual mesh filename=package://atlas/meshes/pelvis.dae scale=1 1 1
- link r_clav: geometry collision mesh filename=package://atlas/meshes/r_clav.stl scale=1 1 1; visual mesh filename=package://atlas/meshes/r_clav.dae scale=1 1 1
- link r_farm: geometry collision mesh filename=package://atlas/meshes/r_farm.stl scale=1 1 1; visual mesh filename=package://atlas/meshes/r_farm.dae scale=1 1 1
- link r_foot: geometry collision mesh filename=package://atlas/meshes/r_foot.stl scale=1 1 1; visual mesh filename=package://atlas/meshes/r_foot.dae scale=1 1 1
- link r_hand: geometry collision mesh filename=package://atlas/meshes/r_hand.stl scale=1 1 1; visual mesh filename=package://atlas/meshes/r_hand.dae scale=1 1 1
- link r_larm: geometry collision mesh filename=package://atlas/meshes/r_larm.stl scale=1 1 1; visual mesh filename=package://atlas/meshes/r_larm.dae scale=1 1 1
- link r_lglut: geometry collision mesh filename=package://atlas/meshes/r_lglut.stl scale=1 1 1; visual mesh filename=package://atlas/meshes/r_lglut.dae scale=1 1 1
- link r_lleg: geometry collision mesh filename=package://atlas/meshes/r_lleg.stl scale=1 1 1; visual mesh filename=package://atlas/meshes/r_lleg.dae scale=1 1 1
- link r_scap: geometry collision mesh filename=package://atlas/meshes/r_scap.stl scale=1 1 1; visual mesh filename=package://atlas/meshes/r_scap.dae scale=1 1 1
- link r_talus: geometry collision mesh filename=package://atlas/meshes/r_talus.stl scale=1 1 1; visual mesh filename=package://atlas/meshes/r_talus.dae scale=1 1 1
- link r_uarm: geometry collision mesh filename=package://atlas/meshes/r_uarm.stl scale=1 1 1; visual mesh filename=package://atlas/meshes/r_uarm.dae scale=1 1 1
- link r_uglut: geometry collision mesh filename=package://atlas/meshes/r_uglut.stl scale=1 1 1; visual mesh filename=package://atlas/meshes/r_uglut.dae scale=1 1 1
- link r_uleg: geometry collision mesh filename=package://atlas/meshes/r_uleg.stl scale=1 1 1; visual mesh filename=package://atlas/meshes/r_uleg.dae scale=1 1 1
- link utorso: geometry collision mesh filename=package://atlas/meshes/utorso.stl scale=1 1 1; visual mesh filename=package://atlas/meshes/utorso.dae scale=1 1 1

Commit message: fix issue #67, imu link offset is wrong.

File: models/drc_robot/model.urdf (robot description, URDF)
Before this commit: robot drc_robot, 40 links, 39 joints
Joints:
- joint imu_joint: origin xyz=0 0 0 rpy=0.05991527603 0 -0.01415 -> xyz=0.05991527603 0 -0.01415 rpy=0 0 0
