Commit message: beginning to fix head imu

File: ros/multisense_sl_description/urdf/multisense_sl.urdf (robot description, URDF)
Before this commit: robot multisense_sl, 11 links, 10 joints
Links:
- added link imu_link, mass 0.1; collision box size=0.01 0.01 0.01; visual box size=0.01 0.01 0.01
Joints:
- added joint imu_joint: type fixed, parent head, child imu_link, origin xyz=0.05991527603 0 -0.01415 rpy=0 0 0
