Commit message: Made best guess on fixes to equalize limits in one case and provide opposite signs in another case

File: ros/atlas_description/urdf/atlas.urdf (robot description, URDF)
Before this commit: robot drc_skeleton, 28 links, 28 joints
Joints:
- joint l_leg_uhz: limit lower=-0.32 upper=1.14 effort=110 velocity=12 -> lower=-0.32 upper=1.14 effort=260 velocity=12
