Commit message: started simple shape approximations for atlas lower leg

File: ros/atlas_description/urdf/atlas_simple_shapes.urdf (robot description, URDF)
Before this commit: robot drc_skeleton, 28 links, 28 joints
Links:
- link l_lleg: geometry collision cylinder length=0.18 radius=0.06; collision cylinder length=0.22 radius=0.06

Commit message: Fix Atlas mesh scaling, issue #275

File: ros/atlas_description/urdf/atlas_simple_shapes.urdf (robot description, URDF)
Before this commit: robot drc_skeleton, 28 links, 28 joints
Links:
- link l_lleg: geometry collision cylinder length=0.40 radius=0.07; visual mesh filename=package://atlas/meshes/l_lleg.dae scale=1.0 1.0 1.0
- link l_uleg: geometry collision cylinder length=0.10 radius=0.1; collision cylinder length=0.15 radius=0.07
- link pelvis: geometry collision box size=0.1 0.15 0.2; collision cylinder length=0.05 radius=0.16
- link r_larm: geometry collision box size=0.135 0.15 0.06; collision cylinder length=0.125 radius=0.045
- link r_lglut: geometry collision cylinder length=0.060306 radius=0.02009687; collision cylinder length=0.12 radius=0.02
- link r_lleg: geometry collision cylinder length=0.40 radius=0.07; visual mesh filename=package://atlas/meshes/r_lleg.dae scale=1.0 1.0 1.0
- link r_uarm: geometry collision box size=0.04 0.07 0.13; collision cylinder length=0.125 radius=0.045
- link r_uglut: geometry collision cylinder length=0.078396 radius=0.019096; collision cylinder length=0.080842 radius=0.019841
- link r_uleg: geometry collision cylinder length=0.10 radius=0.1; collision cylinder length=0.15 radius=0.07
