Commit message: RobotiQ hand model with joint coupling (note that there are some missing joints.

File: robotiq_hand_description/urdf/robotiq_hand.urdf.xacro (robot description, xacro)
@@ -113,7 +113,224 @@
         <mass value="0.03354"/>
         <inertia ixx="0.00000305151" ixy="0.00000089792" ixz="0.00000000249" iyy="0.00001427978" iyz="-0.00000001191" izz="0.00001264126"/>
-    </inertial>
+      </inertial>
     </link>
     <gazebo reference="${prefix}link_3">
+      <mu1>1.1</mu1>
+      <mu2>1.1</mu2>
+    </gazebo>
+    <!-- Link proximal actuating hinge -->
+    <link name="${prefix}link_proximal_actuating_hinge">
+      <visual>
+        <origin rpy="0 0 0" xyz="0 0 0"/>
+        <geometry>
+          <box size="0.03 .0075 .002"/>
+        </geometry>
+      </visual>
+      <collision>
+        <origin rpy="0 0 0" xyz="0 0 0"/>
+         <geometry>
+          <box size="0.03 .0075 .002"/>
+        </geometry>
+      </collision>
+      <inertial>
+        <origin rpy="0 0 0" xyz="0 0 0"/>
+        <mass value="0.047"/>
+        <inertia ixx="0.00000499332" ixy="0.00000091312" ixz="-0.00000000120" iyy  ="0.00006434531" iyz="-0.00000000007" izz="0.00006061917"/>
+      </inertial>
+    </link>
+    <!-- Link 2 -->
+    <gazebo reference="${prefix}link_proximal_actuating_hinge">
+      <mu1>1.1</mu1>
+      <mu2>1.1</mu2>
+    </gazebo>
+    <!-- Link paraproximal actuating hinge -->
+    <link name="${prefix}link_paraproximal_actuating_hinge">
+      <visual>
+        <origin rpy="0 0 0" xyz="0 0 0"/>
+        <geometry>
+          <box size="0.03 .0075 .002"/>
+        </geometry>
+      </visual>
+      <collision>
+        <origin rpy="0 0 0" xyz="0 0 0"/>
+         <geometry>
+          <box size="0.03 .0075 .002"/>
+        </geometry>
+      </collision>
+      <inertial>
+        <origin rpy="0 0 0" xyz="0 0 0"/>
+        <mass value="0.047"/>
+        <inertia ixx="0.00000499332" ixy="0.00000091312" ixz="-0.00000000120" iyy  ="0.00006434531" iyz="-0.00000000007" izz="0.00006061917"/>
+      </inertial>
+    </link>
+    <gazebo reference="${prefix}link_paraproximal_actuating_hinge">
+      <mu1>1.1</mu1>
+      <mu2>1.1</mu2>
+    </gazebo>
+    <!-- Link proximal actuating bar -->
+    <link name="${prefix}link_proximal_actuating_bar">
+      <visual>
+        <origin rpy="0 0 0" xyz="0 0 0"/>
+        <geometry>
+          <box size="0.053578 .0075 .002"/>
+        </geometry>
+      </visual>
+      <collision>
+        <origin rpy="0 0 0" xyz="0 0 0"/>
+         <geometry>
+          <box size="0.053578 .0075 .002"/>
+        </geometry>
+      </collision>
+      <inertial>
+        <origin rpy="0 0 0" xyz="0 0 0"/>
+        <mass value="0.047"/>
+        <inertia ixx="0.00000499332" ixy="0.00000091312" ixz="-0.00000000120" iyy  ="0.00006434531" iyz="-0.00000000007" izz="0.00006061917"/>
+      </inertial>
+    </link>
+    <gazebo reference="${prefix}link_proximal_actuating_bar">
+      <mu1>1.1</mu1>
+      <mu2>1.1</mu2>
+    </gazebo>
+    <!-- Link paraproximal bar -->
+    <link name="${prefix}link_paraproximal_bar">
+      <visual>
+        <origin rpy="0 0 0" xyz="0 0 0"/>
+        <geometry>
+          <box size="0.05715 .0075 .002"/>
+        </geometry>
+      </visual>
+      <collision>
+        <origin rpy="0 0 0" xyz="0 0 0"/>
+         <geometry>
+          <box size="0.05715 .0075 .002"/>
+        </geometry>
+      </collision>
+      <inertial>
+        <origin rpy="0 0 0" xyz="0 0 0"/>
+        <mass value="0.047"/>
+        <inertia ixx="0.00000499332" ixy="0.00000091312" ixz="-0.00000000120" iyy  ="0.00006434531" iyz="-0.00000000007" izz="0.00006061917"/>
+      </inertial>
+    </link>
+    <gazebo reference="${prefix}link_paraproximal_bar">
+      <mu1>1.1</mu1>
+      <mu2>1.1</mu2>
+    </gazebo>
+    <!-- Link median actuating hinge -->
+    <link name="${prefix}link_median_actuating_hinge">
+      <visual>
+        <origin rpy="0 0 0" xyz="0 0 0"/>
+        <geometry>
+          <box size=".02 .02 .002"/>
+        </geometry>
+      </visual>
+      <collision>
+        <origin rpy="0 0 0" xyz="0 0 0"/>
+         <geometry>
+          <box size=".02 0.2 0.002"/>
+        </geometry>
+      </collision>
+      <inertial>
+        <origin rpy="0 0 0" xyz="0 0 0"/>
+        <mass value="0.047"/>
+        <inertia ixx="0.00000499332" ixy="0.00000091312" ixz="-0.00000000120" iyy  ="0.00006434531" iyz="-0.00000000007" izz="0.00006061917"/>
+      </inertial>
+    </link>
+    <gazebo reference="${prefix}link_median_actuating_hinge">
+      <mu1>1.1</mu1>
+      <mu2>1.1</mu2>
+    </gazebo>
+    <!-- Link median bar -->
+    <link name="${prefix}link_median_bar">
+      <visual>
+        <origin rpy="0 0 0" xyz="0 0 0"/>
+        <geometry>
+          <box size="0.0381 .0075 .002"/>
+        </geometry>
+      </visual>
+      <collision>
+        <origin rpy="0 0 0" xyz="0 0 0"/>
+         <geometry>
+          <box size="0.0381 .0075 .002"/>
+        </geometry>
+      </collision>
+      <inertial>
+        <origin rpy="0 0 0" xyz="0 0 0"/>
+        <mass value="0.047"/>
+        <inertia ixx="0.00000499332" ixy="0.00000091312" ixz="-0.00000000120" iyy  ="0.00006434531" iyz="-0.00000000007" izz="0.00006061917"/>
+      </inertial>
+    </link>
+    <gazebo reference="${prefix}link_median_bar">
+      <mu1>1.1</mu1>
+      <mu2>1.1</mu2>
+    </gazebo>
+    <!-- Link paramedian hinge -->
+    <link name="${prefix}link_paramedian_hinge">
+      <visual>
+        <origin rpy="0 0 0" xyz="0 0 0"/>
+        <geometry>
+          <box size=".02 .02 .002"/>
+        </geometry>
+      </visual>
+      <collision>
+        <origin rpy="0 0 0" xyz="0 0 0"/>
+         <geometry>
+          <box size=".02 0.2 0.002"/>
+        </geometry>
+      </collision>
+      <inertial>
+        <origin rpy="0 0 0" xyz="0 0 0"/>
+        <mass value="0.047"/>
+        <inertia ixx="0.00000499332" ixy="0.00000091312" ixz="-0.00000000120" iyy  ="0.00006434531" iyz="-0.00000000007" izz="0.00006061917"/>
+      </inertial>
+    </link>
+    <gazebo reference="${prefix}link_paramedian_hinge">
+      <mu1>1.1</mu1>
+      <mu2>1.1</mu2>
+    </gazebo>
+    <!-- Link median bar underactuated -->
+    <link name="${prefix}link_median_bar_underactuated">
+      <visual>
+        <origin rpy="0 0 0" xyz="0 0 0"/>
+        <geometry>
+          <box size="0.0381 .0075 .002"/>
+        </geometry>
+      </visual>
+      <collision>
+        <origin rpy="0 0 0" xyz="0 0 0"/>
+         <geometry>
+          <box size="0.0381 .0075 .002"/>
+        </geometry>
+      </collision>
+      <inertial>
+        <origin rpy="0 0 0" xyz="0 0 0"/>
+        <mass value="0.047"/>
+        <inertia ixx="0.00000499332" ixy="0.00000091312" ixz="-0.00000000120" iyy  ="0.00006434531" iyz="-0.00000000007" izz="0.00006061917"/>
+      </inertial>
+    </link>
+    <gazebo reference="${prefix}link_median_bar_underactuated">
+      <mu1>1.1</mu1>
+      <mu2>1.1</mu2>
+    </gazebo>
+    <!-- Link paradistal hinge -->
+    <link name="${prefix}link_paradistal_hinge">
+      <visual>
+        <origin rpy="0 0 0" xyz="0 0 0"/>
+        <geometry>
+          <box size=".02 .02 .002"/>
+        </geometry>
+      </visual>
+      <collision>
+        <origin rpy="0 0 0" xyz="0 0 0"/>
+         <geometry>
+          <box size=".02 0.2 0.002"/>
+        </geometry>
+      </collision>
+      <inertial>
+        <origin rpy="0 0 0" xyz="0 0 0"/>
+        <mass value="0.047"/>
+        <inertia ixx="0.00000499332" ixy="0.00000091312" ixz="-0.00000000120" iyy  ="0.00006434531" iyz="-0.00000000007" izz="0.00006061917"/>
+      </inertial>
+    </link>
+    <gazebo reference="${prefix}link_paradistal_hinge">
       <mu1>1.1</mu1>
       <mu2>1.1</mu2>
@@ -121,4 +338,103 @@
     <!-- End of link list -->
     <!-- Joint list -->
+    <!-- Joint proximal actuating hinge -->
+    <joint name="${prefix}joint_proximal_actuating_hinge" type="revolute">
+      <parent link="${prefix}link_0"/>
+      <child link="${prefix}link_proximal_actuating_hinge"/>
+      <axis xyz="0 0 1"/>
+      <origin rpy="0 0 1.051" xyz="-0.0071 -0.012 0.01"/>
+      <limit effort="100" lower="0" upper="3.1416" velocity="100"/>
+    </joint>
+    <gazebo reference="${prefix}joint_proximal_actuating_hinge">
+      <implicitSpringDamper>1</implicitSpringDamper>
+    </gazebo>
+    <!-- Joint paraproximal actuating hinge -->
+    <joint name="${prefix}joint_paraproximal_actuating_hinge" type="revolute">
+      <parent link="${prefix}link_0"/>
+      <child link="${prefix}link_paraproximal_actuating_hinge"/>
+      <axis xyz="0 0 1"/>
+      <origin rpy="0 0 1.051" xyz="-0.0071 -0.012 -0.01"/>
+      <limit effort="100" lower="0" upper="3.1416" velocity="100"/>
+    </joint>
+    <gazebo reference="${prefix}joint_paraproximal_actuating_hinge">
+      <implicitSpringDamper>1</implicitSpringDamper>
+    </gazebo>
+    <!-- Joint proximal actuating bar -->
+    <joint name="${prefix}joint_proximal_actuating_bar" type="revolute">
+      <parent link="${prefix}link_proximal_actuating_hinge"/>
+      <child link="${prefix}link_proximal_actuating_bar"/>
+      <axis xyz="0 0 1"/>
+      <origin rpy="0 0 -1.28" xyz="-0.0067 -0.0257 0"/>
+      <limit effort="100" lower="0" upper="3.1416" velocity="100"/>
+    </joint>
+    <gazebo reference="${prefix}joint_proximal_actuating_bar">
+      <implicitSpringDamper>1</implicitSpringDamper>
+    </gazebo>
+    <!-- Joint paraproximal bar -->
+    <joint name="${prefix}joint_paraproximal_bar" type="revolute">
+      <parent link="${prefix}link_paraproximal_actuating_hinge"/>
+      <child link="${prefix}link_paraproximal_bar"/>
+      <axis xyz="0 0 1"/>
+      <origin rpy="0 0 -1.57" xyz="-0.015 -0.029 0"/>
+      <limit effort="100" lower="0" upper="3.1416" velocity="100"/>
+    </joint>
+    <gazebo reference="${prefix}joint_paraproximal_bar">
+      <implicitSpringDamper>1</implicitSpringDamper>
+    </gazebo>
+    <!-- Joint median actuating hinge -->
+    <joint name="${prefix}joint_median_actuating_hinge" type="revolute">
+      <parent link="${prefix}link_1"/>
+      <child link="${prefix}link_median_actuating_hinge"/>
+      <axis xyz="0 0 1"/>
+      <origin rpy="0 0 -0.52" xyz="0.050 -.028 0.01"/>
+      <limit effort="100" lower="0" upper="3.1416" velocity="100"/>
+    </joint>
+    <gazebo reference="${prefix}joint_median_actuating_hinge">
+      <implicitSpringDamper>1</implicitSpringDamper>
+    </gazebo>
+    <!-- Joint paramedian hinge -->
+    <joint name="${prefix}joint_paramedian_hinge" type="revolute">
+      <parent link="${prefix}link_1"/>
+      <child link="${prefix}link_paramedian_hinge"/>
+      <axis xyz="0 0 1"/>
+      <origin rpy="0 0 -0.52" xyz="0.050 -.028 -0.01"/>
+      <limit effort="100" lower="0" upper="3.1416" velocity="100"/>
+    </joint>
+    <gazebo reference="${prefix}joint_paramedian_hinge">
+      <implicitSpringDamper>1</implicitSpringDamper>
+    </gazebo>
+    <!-- Joint median actuating hinge median bar -->
+    <joint name="${prefix}joint_median_actuating_hinge_median_bar" type="revolute">
+      <parent link="${prefix}link_median_actuating_hinge"/>
+      <child link="${prefix}link_median_bar"/>
+      <axis xyz="0 0 1"/>
+      <origin rpy="0 0 0.29" xyz="0.019 -0.02381 0"/>
+      <limit effort="100" lower="0" upper="3.1416" velocity="100"/>
+    </joint>
+    <gazebo reference="${prefix}joint_median_actuating_hinge_median_bar">
+      <implicitSpringDamper>1</implicitSpringDamper>
+    </gazebo>
+    <!-- Joint paradistal hinge -->
+    <joint name="${prefix}joint_paradistal_hinge" type="revolute">
+      <parent link="${prefix}link_2"/>
+      <child link="${prefix}link_paradistal_hinge"/>
+      <axis xyz="0 0 1"/>
+      <origin rpy="0 0 0" xyz="0.039 0 0.01"/>
+      <limit effort="100" lower="0" upper="3.1416" velocity="100"/>
+    </joint>
+    <gazebo reference="${prefix}joint_paradistal_hinge">
+      <implicitSpringDamper>1</implicitSpringDamper>
+    </gazebo>
+    <!-- Joint paramedian hinge median bar underactuated -->
+    <joint name="${prefix}joint_paramedian_hinge_median_bar_underactuated" type="revolute">
+      <parent link="${prefix}link_paramedian_hinge"/>
+      <child link="${prefix}link_median_bar_underactuated"/>
+      <axis xyz="0 0 1"/>
+      <origin rpy="0 0 0" xyz="0.01786 -0.011905 0"/>
+      <limit effort="100" lower="0" upper="3.1416" velocity="100"/>
+    </joint>
+    <gazebo reference="${prefix}joint_paramedian_hinge_median_bar_underactuated">
+      <implicitSpringDamper>1</implicitSpringDamper>
+    </gazebo>
     <!-- Joint 1 -->
     <joint name="${prefix}joint_1" type="revolute">
