Commit message: adding new v4 and new v5

File: atlas_description/urdf/atlas_v4_raw.urdf (robot description, URDF)
Before this commit: robot drc_skeleton, 34 links, 34 joints
Links:
- removed link l_situational_awareness_camera_link
- removed link l_situational_awareness_camera_optical_frame
- removed link r_situational_awareness_camera_link
- removed link r_situational_awareness_camera_optical_frame
- removed link rear_situational_awareness_camera_link
- removed link rear_situational_awareness_camera_optical_frame
- added link head, mass 3.751
- link l_clav: geometry 
- link l_farm: geometry 
- link l_foot: geometry 
- link l_hand: geometry 
- link l_larm: geometry 
- link l_lglut: geometry 
- link l_lleg: geometry 
- link l_scap: geometry 
- link l_talus: geometry 
- link l_uarm: geometry 
- link l_uglut: geometry 
- link l_uleg: geometry 
- link ltorso: geometry 
- link mtorso: geometry 
- link pelvis: geometry 
- link r_clav: geometry 
- link r_farm: geometry 
- link r_foot: geometry 
- link r_hand: geometry 
- link r_larm: geometry 
- link r_lglut: geometry 
- link r_lleg: geometry 
- link r_scap: geometry 
- link r_talus: geometry 
- link r_uarm: geometry 
- link r_uglut: geometry 
- link r_uleg: geometry 
- link utorso: geometry 
Joints:
- removed joint l_situational_awareness_camera_joint
- removed joint l_situational_awareness_camera_optical_frame_joint
- removed joint r_situational_awareness_camera_joint
- removed joint r_situational_awareness_camera_optical_frame_joint
- removed joint rear_situational_awareness_camera_joint
- removed joint rear_situational_awareness_camera_optical_frame_joint
