Commit message: Simple shapes for the new arms.

File: atlas_description/urdf/atlas_v4_simple_shapes.urdf (robot description, URDF)
Before this commit: robot drc_skeleton, 34 links, 34 joints
Links:
- link l_clav: geometry collision box size=0.02 0.029 0.015; collision box size=0.02 0.19 0.072
- link l_farm: geometry collision box size=0.145 0.115 0.12; collision cylinder length=0.145 radius=0.055
- link l_hand: geometry collision box size=0.14 0.09 0.06; collision cylinder length=0.012 radius=0.048
- link l_larm: geometry collision box size=0.025 0.125 0.075; collision cylinder length=0.04 radius=0.041
- link l_scap: geometry collision box size=0.15 0.15 0.06; collision cylinder length=0.05 radius=0.04
- link l_uarm: geometry collision box size=0.05 0.07 0.15; collision cylinder length=0.11 radius=0.065
- link r_clav: geometry collision box size=0.02 0.029 0.015; collision box size=0.02 0.19 0.072
- link r_farm: geometry collision box size=0.145 0.115 0.12; collision cylinder length=0.145 radius=0.055
- link r_hand: geometry collision box size=0.14 0.09 0.06; collision cylinder length=0.012 radius=0.048
- link r_larm: geometry collision box size=0.025 0.125 0.075; collision cylinder length=0.04 radius=0.041
- link r_scap: geometry collision box size=0.15 0.15 0.06; collision cylinder length=0.05 radius=0.04
- link r_uarm: geometry collision box size=0.05 0.07 0.15; collision cylinder length=0.11 radius=0.065
